File: pcb/SCuSA_A1/SCuSA.kicad_pcb (KiCad board)
At the start: 2 copper layers, 56 x 68 mm, 65 parts, among them J101 USB4135-GF-A, J102 JST_S2B-PH-K-x, J103 Binding_Post_PK4_Red, J104 Binding_Post_PK4_Black, J105 SMA_Straight_Jack_Female, J107 77311-118-02LF, J108 77311-118-02LF, Q101 DMN2041LSD, SW101 JS202011CQN, SW102 JS202011CQN, U101 MCP73832T-2ACI/OT, U102 BQ29700DSER, U103 TLV803EA30DBZR, U104 LM27762, U105 AD8410AWBRZ, U106 AD8655ARZ

Commit message: Edit PCB layout
Parts:
- added H101: MountingHole, MountingHole:MountingHole_3.2mm_M3_DIN965, F.Cu at (159.5, 65.5)
- added H102: MountingHole, MountingHole:MountingHole_3.2mm_M3_DIN965, F.Cu at (115.5, 65.5)
- added H103: MountingHole, MountingHole:MountingHole_3.2mm_M3_DIN965, F.Cu at (115.5, 100.5)
- added H104: MountingHole, MountingHole:MountingHole_3.2mm_M3_DIN965, F.Cu at (159.5, 100.5)
- added R120: 0R,0603, Resistor_SMD:R_0603_1608Metric_Pad0.98x0.95mm_HandSolder, F.Cu at (134.5, 88.5)
- JP101: value SolderJumper_2_Bridged -> SolderJumper_2_Open; footprint Jumper:SolderJumper-2_P1.3mm_Bridged_Pad1.0x1.5mm -> Jumper:SolderJumper-2_P1.3mm_Open_TrianglePad1.0x1.5mm
- R103: value 2k,0603 -> 10k,0603
- moved TP106 51.2 mm to (152.0, 86.0), turned to 90 degrees
- moved TP104 45.9 mm to (142.0, 93.0)
- moved TP103 44.2 mm to (140.0, 101.5)
- moved TP108 43.3 mm to (156.0, 82.5), turned to 90 degrees
- moved TP101 35.4 mm to (134.5, 101.5)
- moved TP105 34.5 mm to (135.0, 85.5)
- moved J101 33.4 mm to (117.4, 74.8), turned to -90 degrees
- moved R101 32.5 mm to (119.2, 72.0)
- moved R107 32.2 mm to (114.5, 89.5)
- moved TP102 32.2 mm to (129.0, 101.5)
- moved TP107 32.1 mm to (156.0, 89.0), turned to 90 degrees
- moved R117 30.0 mm to (128.0, 81.0), turned to 180 degrees
- moved R102 29.8 mm to (120.2, 74.8), turned to 0 degrees
- moved J102 29.7 mm to (121.5, 102.0), turned to 0 degrees
- moved R108 28.3 mm to (114.5, 96.5)
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Connections:
- JP101 pad 1: /VBat_SW -> GND
- JP101 pad 2: Net-(JP101-B) -> /Cell-
- U104 pad 12: Net-(JP101-B) -> Net-(U104-EN+)
Other:
- board size 56 x 68 mm -> 51 x 42 mm

Commit message: Edit PCB layout
Parts:
- moved R111 3.47 mm to (131.1, 85.2), turned to 0 degrees
- moved R107 2.20 mm to (116.7, 89.5), turned to 180 degrees
- moved R108 2.20 mm to (116.7, 96.5)
- moved R101 1.61 mm to (120.2, 73.3), turned to 0 degrees
- moved R104 0.99 mm to (124.0, 79.1), turned to 180 degrees
- moved U102 0.97 mm to (123.8, 93.8)
- moved C103 0.43 mm to (124.5, 91.8)
- moved R105 0.35 mm to (124.5, 90.2)
- moved D101 0.35 mm to (120.4, 79.0)
- moved R106 0.32 mm to (122.0, 91.0)
- moved FB101 0.25 mm to (131.5, 97.5)
- moved JP101 0.23 mm to (123.5, 98.5), turned to -90 degrees
- moved U103 0.20 mm to (132.0, 80.3)
- moved U105 0.18 mm to (137.6, 78.5)
- moved R112 0.14 mm to (133.7, 94.6)
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Routing:
- net /Cell-: track 0.00 -> 17.0 mm
- net Net-(Q101A-G1): track 0.00 -> 16.9 mm
- net Net-(Q101B-G2): track 0.00 -> 14.7 mm, vias 0 -> 2
- net /PGOOD: track 0.00 -> 12.0 mm, vias 0 -> 2
- net /VBus: track 0.00 -> 8.07 mm
- net Net-(F101-Pad1): track 0.00 -> 7.75 mm
- net Net-(D101-K): track 0.00 -> 7.66 mm
- net Net-(U104-FB+): track 0.00 -> 7.61 mm
- net Net-(U104-EN+): track 0.00 -> 5.93 mm
- net Net-(U104-FB-): track 0.00 -> 5.24 mm
- net Net-(U104-EN-): track 0.00 -> 4.15 mm
- net Net-(Q101A-D1-Pad7): track 0.00 -> 3.81 mm
- net Net-(U102-BAT): track 0.00 -> 3.13 mm
- net +3V3: track 0.00 -> 2.91 mm
- net GND: track 0.00 -> 2.78 mm, vias 0 -> 2
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