File: pcb/SCuSA_A1/SCuSA.kicad_sch (KiCad schematic)
At the start: 74 parts, among them J101 USB4135-GF-A, J102 JST_S2B-PH-K-x, J103 Binding_Post_PKI_10_A_Au, J104 Binding_Post_PKI_10_A_Au, J105 SMA_Straight_Jack_Female, J107 77311-118-02LF, J108 77311-118-02LF, Q101 DMN2041LSD, SW101 JS202011CQN, SW102 JS202011CQN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

Commit message: Fix errors, edit PCB layout
Parts:
- added C120: 100nF,16V,X7R,0603, Capacitor_SMD:C_0603_1608Metric_Pad1.08x0.95mm_HandSolder, symbol Capacitor_User:100nF,16V,X7R,0603
- C101, C102: footprint Capacitor_SMD:C_0603_1608Metric_Pad1.08x0.95mm_HandSolder -> Capacitor_SMD:C_0805_2012Metric_Pad1.18x1.45mm_HandSolder; symbol Capacitor_User:1uF,16V,X7R,0603 -> Capacitor_User:4.7uF,25V,X7R,0805; Pretty Value 1 1μF, 16V -> 4.7μF, 25V; Pretty Value 2 X7R, 0603 -> X7R, 0805
Connections:
- net GND: now also U103.2 (GND), C120.1; no longer U103.1 (GND)
- net VBat_SW: now also C120.2
- net at D102.1 (K): now also U103.1 (~{RESET}); no longer U103.2 (~{RESET})
Changed lines of the file:
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@@
   (junction (at 198.12 43.18) (diameter 0) (color 0 0 0 0)
   )
+  (junction (at 24.13 170.18) (diameter 0) (color 0 0 0 0)
+  )
   (junction (at 46.99 27.94) (diameter 0) (color 0 0 0 0)
   )
@@
   (junction (at 260.35 114.3) (diameter 0) (color 0 0 0 0)
   )
+  (junction (at 41.91 187.96) (diameter 0) (color 0 0 0 0)
+  )
   (junction (at 90.17 142.24) (diameter 0) (color 0 0 0 0)
   )
@@
     (stroke (width 0) (type default))
   )
+  (wire (pts (xy 24.13 187.96) (xy 41.91 187.96))
+    (stroke (width 0) (type default))
+  )
   (wire (pts (xy 227.33 29.21) (xy 227.33 43.18))
     (stroke (width 0) (type default))
@@
     (stroke (width 0) (type default))
   )
+  (wire (pts (xy 24.13 182.88) (xy 24.13 187.96))
+    (stroke (width 0) (type default))
+  )
   (wire (pts (xy 260.35 114.3) (xy 265.43 114.3))
     (stroke (width 0) (type default))
@@
     (stroke (width 0) (type default))
   )
+  (wire (pts (xy 24.13 177.8) (xy 24.13 170.18))
+    (stroke (width 0) (type default))
+  )
   (wire (pts (xy 204.47 149.86) (xy 201.93 149.86))
     (stroke (width 0) (type default))
@@
     )
   )
+  (symbol (lib_id "Capacitor_User:100nF,16V,X7R,0603") (at 24.13 180.34 180) (unit 1)
+    (in_bom yes) (on_board yes) (dnp yes) (fields_autoplaced)
+    (property "Reference" "C120" (at 26.67 177.7936 0)
+      (effects (font (size 1.27 1.27)) (justify right))
+    )
+    (property "Value" "100nF,16V,X7R,0603" (at 21.59 175.26 0)
+      (effects (font (size 1.27 1.27)) (justify left) hide)
+    )
+    (property "Footprint" "Capacitor_SMD:C_0603_1608Metric_Pad1.08x0.95mm_HandSolder" (at 22.86 168.91 0)
+      (effects (font (size 1.27 1.27)) hide)
+    )
+    (property "Datasheet" "~" (at 24.13 180.34 0)
+      (effects (font (size 1.27 1.27)) hide)
+    )
+    (property "Pretty Value 1" "100nF, 16V" (at 26.67 180.3336 0)
+      (effects (font (size 1.27 1.27)) (justify right))
+    )
+    (property "Pretty Value 2" "X7R, 0603" (at 26.67 182.8736 0)
+      (effects (font (size 1.27 1.27)) (justify right))
+    )
+    (pin "1")
+    (pin "2")
+    (instances
+      (project "SCuSA"
+        (path "/7c524ebf-103a-4dc7-9ca9-e5a941b364b9"
+          (reference "C120") (unit 1)
+        )
+      )
+    )
+  )
   (symbol (lib_id "Resistor_User:68k,0603") (at 90.17 120.65 0) (unit 1)
     (in_bom yes) (on_board yes) (dnp no) (fields_autoplaced)
@@
     )
   )
-  (symbol (lib_id "Capacitor_User:1uF,16V,X7R,0603") (at 69.85 39.37 0) (unit 1)
+  (symbol (lib_id "Capacitor_User:4.7uF,25V,X7R,0805") (at 69.85 39.37 0) (unit 1)
     (in_bom yes) (on_board yes) (dnp no) (fields_autoplaced)
     (property "Reference" "C101" (at 72.39 36.8363 0)
@@
       (effects (font (size 1.27 1.27)) (justify left) hide)
     )
-    (property "Footprint" "Capacitor_SMD:C_0603_1608Metric_Pad1.08x0.95mm_HandSolder" (at 71.12 50.8 0)
+    (property "Footprint" "Capacitor_SMD:C_0805_2012Metric_Pad1.18x1.45mm_HandSolder" (at 71.12 50.8 0)
       (effects (font (size 1.27 1.27)) hide)
     )
@@
       (effects (font (size 1.27 1.27)) hide)
     )
-    (property "Pretty Value 1" "1μF, 16V" (at 72.39 39.3763 0)
+    (property "Pretty Value 1" "4.7μF, 25V" (at 72.39 39.3763 0)
       (effects (font (size 1.27 1.27)) (justify left))
     )
-    (property "Pretty Value 2" "X7R, 0603" (at 72.39 41.9163 0)
+    (property "Pretty Value 2" "X7R, 0805" (at 72.39 41.9163 0)
       (effects (font (size 1.27 1.27)) (justify left))
     )
@@
   )
   (symbol (lib_id "Power_Supervisor_User:TLV803EA30DBZR") (at 41.91 180.34 0) (unit 1)
-    (in_bom yes) (on_board yes) (dnp no) (fields_autoplaced)
-    (property "Reference" "U103" (at 38.1 179.07 0)
+    (in_bom yes) (on_board yes) (dnp no)
+    (property "Reference" "U103" (at 48.26 173.99 0)
       (effects (font (size 1.27 1.27)) (justify right))
     )
-    (property "Value" "TLV803EA30DBZR" (at 38.1 181.61 0)
+    (property "Value" "TLV803EA30DBZR" (at 59.69 186.69 0)
       (effects (font (size 1.27 1.27)) (justify right))
     )
@@
     )
   )
-  (symbol (lib_id "Capacitor_User:1uF,16V,X7R,0603") (at 110.49 39.37 0) (unit 1)
+  (symbol (lib_id "Capacitor_User:4.7uF,25V,X7R,0805") (at 110.49 39.37 0) (unit 1)
     (in_bom yes) (on_board yes) (dnp no) (fields_autoplaced)
     (property "Reference" "C102" (at 113.03 36.8363 0)
@@
       (effects (font (size 1.27 1.27)) (justify left) hide)
     )
-    (property "Footprint" "Capacitor_SMD:C_0603_1608Metric_Pad1.08x0.95mm_HandSolder" (at 111.76 50.8 0)
+    (property "Footprint" "Capacitor_SMD:C_0805_2012Metric_Pad1.18x1.45mm_HandSolder" (at 111.76 50.8 0)
       (effects (font (size 1.27 1.27)) hide)
     )
@@
       (effects (font (size 1.27 1.27)) hide)
     )
-    (property "Pretty Value 1" "1μF, 16V" (at 113.03 39.3763 0)
+    (property "Pretty Value 1" "4.7μF, 25V" (at 113.03 39.3763 0)
       (effects (font (size 1.27 1.27)) (justify left))
     )
-    (property "Pretty Value 2" "X7R, 0603" (at 113.03 41.9163 0)
+    (property "Pretty Value 2" "X7R, 0805" (at 113.03 41.9163 0)
       (effects (font (size 1.27 1.27)) (justify left))
     )
