File: pcb/SCuSA_B1/SCuSA.kicad_pcb (KiCad board)
At the start: 2 copper layers, 51 x 42 mm, 65 parts, among them J101 USB4135-GF-A, J102 JST_S2B-PH-SM4-x, J103 Binding_Post_PKI_10_A_Au, J104 Binding_Post_PKI_10_A_Au, J105 SMA_Straight_Jack_Female, J107 77311-118-02LF, J108 77311-118-02LF, Q101 DMN2041LSD, SW101 JS202011CQN, SW102 JS202011CQN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

Commit message: Edit PCB layout
Parts:
- removed R110: 0R,0603, Resistor_SMD:R_0603_1608Metric_Pad0.98x0.95mm_HandSolder
- added JP101: SolderJumper_2_Open, Jumper:SolderJumper-2_P1.3mm_Open_TrianglePad1.0x1.5mm, F.Cu at (116.6, 92.8)
- moved J102 0.50 mm to (124.9, 98.7)
Routing:
- net Net-(Q101A-G1): track 17.8 -> 20.0 mm
- net GND: track 64.9 -> 64.7 mm, vias 21 -> 20
- net /VBat_SW: vias 2 -> 1
Other:
- board text added: "+ -"
- board text added: "Charge"
- board text added: "Common Mode Voltage Range -2 V to +70 V"
- board text added: "Low Bat."
- board text added: "Offset +←→-"
- board text added: "Offset On/Off"
- board text added: "Rev B1, by fl0m0"
- board text added: "SCuSA"
- board text added: "Scope Current Sense Amplifier"
- board text removed: "*"
- board text removed: "**"
- board text removed: "+"
- board text removed: "-"
- board text removed: "Low Bat"
- board text removed: "Max. -2V to +70V"
- board text removed: "PWR"
- board text removed: "SCuSA Scope Current Sense Amplifier Rev B1, by fl0m0"
- board text removed: "Trim +←→-"
- board text removed: "Trim On/Off"

Commit message: PCB RevB1
Parts:
- moved R106 0.59 mm to (121.4, 91.7)
- moved C103 0.55 mm to (124.2, 91.3)
- moved R105 0.55 mm to (124.2, 89.7)
- moved U102 0.55 mm to (123.5, 93.3)
Routing:
- net /Cell-: track 21.9 -> 20.1 mm
- net /VBat: track 27.7 -> 26.0 mm
- net Net-(Q101A-G1): track 20.0 -> 19.3 mm
